Commit message: Fixed urdf modell.

File: urdf/robotino.urdf (robot description, URDF)
Before this commit: robot robotino, 9 links, 8 joints
Links:
- removed link anglebracketusb_link
- removed link camera_link
- removed link command_bridge_link
- link base_link: mass 20 -> None
- link uwb_reciever_link: mass None -> 0.00001
Joints:
- removed joint anglebracketusb_joint
- removed joint camera_joint
- removed joint command_bridge_joint
- joint laser_joint: origin xyz=-0.05 0 0.225 rpy=0 0 0 -> xyz=0.0 0 0.225 rpy=0 0 0
- joint uwb_reciever_joint: origin xyz=0.05 0 0.2 rpy=0 0 0 -> xyz=0.05 0 0.15 rpy=0 0 0

File: urdf/robotino.urdf.xacro (robot description, xacro)
@@ -1,7 +1,7 @@
 <?xml version="1.0"?>
-<robot name="robotino">
+<robot name="robotino" xmlns:xacro="http://www.ros.org/wiki/xacro">
   <!-- Include files -->
-  <include filename="$(find ro_slam_with_uwb)/urdf/robotino_body.xacro"/>
-  <include filename="$(find ro_slam_with_uwb)/urdf/robotino_hardware.xacro"/>
-  <robotino_body />
+  <xacro:include filename="$(find ro_slam_with_uwb)/urdf/robotino_body.xacro"/>
+  <xacro:include filename="$(find ro_slam_with_uwb)/urdf/robotino_hardware.xacro"/>
+  <xacro:robotino_body />
 </robot>

File: urdf/robotino_body.xacro (robot description, xacro)
@@ -1,11 +1,12 @@
 <?xml version="1.0"?>
-<robot>
-  <property name="M_PI" value="3.14159"/>
-  <property name="M_SCALE" value="0.01"/>
-  <property name="BASE_RADIUS" value="0.18"/>
-  <property name="BASE_HEIGHT" value="0.05"/>
-  <property name="BASE_MASS" value="20"/>
-  <macro name="robotino_body">
+<robot xmlns:xacro="http://www.ros.org/wiki/xacro">
+  <xacro:property name="M_PI" value="3.14159"/>
+  <xacro:property name="M_SCALE" value="0.01"/>
+  <xacro:property name="BASE_RADIUS" value="0.18"/>
+  <xacro:property name="BASE_HEIGHT" value="0.05"/>
+  <xacro:property name="BASE_MASS" value="20"/>
+  <xacro:macro name="robotino_body">
   	<link name="base_link">
+      <!--
       <inertial>
         <mass value="${BASE_MASS}" />
@@ -15,4 +16,5 @@
           izz="1.0" />
       </inertial>
+      -->
       <visual>
         <origin xyz="0.01 0 0" rpy="0 0 ${M_PI/2}"/>
@@ -28,32 +30,38 @@
       </collision>
     </link>
-    <wheel name="wheel0" parent="base_link">
+    <xacro:wheel name="wheel0" parent="base_link">
       <origin xyz="0.065 0.11 0.04" rpy="0 0 ${M_PI/3}"/>
       <axis xyz="-1 0 0"/>
-    </wheel>
-    <wheel name="wheel1" parent="base_link">
+    </xacro:wheel>
+    <xacro:wheel name="wheel1" parent="base_link">
       <origin xyz="-0.13 0 0.04" rpy="0 0 0"/>
       <axis xyz="1 0 0"/>
-    </wheel>
-    <wheel name="wheel2" parent="base_link">
+    </xacro:wheel>
+    <xacro:wheel name="wheel2" parent="base_link">
       <origin xyz="0.065 -0.11 0.04" rpy="0 0 -${M_PI/3}"/>
       <axis xyz="-1 0 0"/>
-    </wheel>
+    </xacro:wheel>
+    <!--
     <command_bridge name="command_bridge" parent="base_link">
       <origin xyz="-0.05 0 0.13" rpy="0 0 ${M_PI/2}"/>
     </command_bridge>
+    -->
+    <!--
     <camera name="camera" parent="base_link">
       <origin xyz="0.044 0 0.07" rpy="0 0 ${M_PI/2}"/>
     </camera>
+    -->
+    <!--
     <anglebracketusb name="anglebracketusb" parent="base_link">
       <origin xyz="0.008 0 0.137" rpy="0 0 ${M_PI/2}"/>
     </anglebracketusb>
-    <laser name="laser" parent="base_link">
+    -->
+    <xacro:laser name="laser" parent="base_link">
       <!--origin xyz="-0.022 0 0.232" rpy="0 0 0"/-->
-      <origin xyz="0.1 0 0" rpy="0 0 0"/>
-    </laser>
-    <!--laser name="laser" parent="base_link"-->
-      <!--origin xyz="0.12 0 ${BASE_HEIGHT/2}" rpy="0 0 0"/-->
-    <!--/laser-->
-  </macro>
+      <origin xyz="0.0 0 0.225" rpy="0 0 0"/>
+    </xacro:laser>
+    <xacro:uwb name="uwb_reciever" parent="base_link">
+      <origin xyz="0.05 0 0.15" rpy="0 0 0"/>
+    </xacro:uwb>
+  </xacro:macro>
 </robot>

File: urdf/robotino_hardware.xacro (robot description, xacro)
@@ -1,16 +1,16 @@
 <?xml version="1.0"?>
-<robot>
-  <property name="M_PI" value="3.14159"/>
-  <property name="M_SCALE" value="0.01"/>
-  <property name="HOKUYO_RADIUS" value="0.02"/>
-  <property name="HOKUYO_LENGTH" value="0.07"/>
-  <property name="KINECT_LENGTH" value="0.064"/>
-  <property name="KINECT_WIDTH" value="0.121"/>
-  <property name="KINECT_HEIGHT" value="0.0381"/>
+<robot xmlns:xacro="http://www.ros.org/wiki/xacro">
+  <xacro:property name="M_PI" value="3.14159"/>
+  <xacro:property name="M_SCALE" value="0.01"/>
+  <xacro:property name="HOKUYO_RADIUS" value="0.02"/>
+  <xacro:property name="HOKUYO_LENGTH" value="0.07"/>
+  <xacro:property name="KINECT_LENGTH" value="0.064"/>
+  <xacro:property name="KINECT_WIDTH" value="0.121"/>
+  <xacro:property name="KINECT_HEIGHT" value="0.0381"/>
   <!-- WHEEL -->
-  <macro name="wheel" params="parent name *origin *axis">
+  <xacro:macro name="wheel" params="parent name *origin *axis">
     <joint name="${name}_joint" type="continuous">
-      <insert_block name="origin" />
-      <insert_block name="axis" />
+      <xacro:insert_block name="origin" />
+      <xacro:insert_block name="axis" />
       <parent link="${parent}"/>
       <child link="${name}_link" />
@@ -31,9 +31,9 @@
       </visual>
     </link>
-  </macro>
+  </xacro:macro>
   <!-- COMMAND BRIDGE -->
-  <macro name="command_bridge" params="parent name *origin">
+  <xacro:macro name="command_bridge" params="parent name *origin">
     <joint name="${name}_joint" type="fixed">
-      <insert_block name="origin" />
+      <xacro:insert_block name="origin" />
       <parent link="${parent}"/>
       <child link="${name}_link" />
@@ -54,9 +54,9 @@
       </collision>
     </link>
-  </macro>
+  </xacro:macro>
   <!-- LASER SCANNER -->
-  <macro name="laser" params="parent name *origin">
+  <xacro:macro name="laser" params="parent name *origin">
     <joint name="${name}_joint" type="fixed">
-      <insert_block name="origin" />
+      <xacro:insert_block name="origin" />
       <parent link="${parent}"/>
       <child link="${name}_link" />
@@ -83,9 +83,25 @@
       </collision>
     </link>
-  </macro>
+  </xacro:macro>
+  <!-- UWB RECIEVER -->
+  <xacro:macro name="uwb" params="parent name *origin">
+    <joint name="${name}_joint" type="fixed">
+      <xacro:insert_block name="origin" />
+      <parent link="${parent}"/>
+      <child link="${name}_link" />
+    </joint>
+    <link name="${name}_link">
+      <inertial>
+        <mass value="0.00001" />
+        <origin xyz="0 0 0" />
+        <inertia ixx="1.0" ixy="0.0" ixz="0.0" iyy="1.0" iyz="0.0" izz="1.0" />
+      </inertial>
+    </link>
+  </xacro:macro>
   <!-- Camera -->
-  <macro name="camera" params="parent name *origin">
+  <!--
+  <xacro:macro name="camera" params="parent name *origin">
     <joint name="${name}_joint" type="fixed">
-      <insert_block name="origin" />
+      <xacro:insert_block name="origin" />
       <parent link="${parent}"/>
       <child link="${name}_link" />
@@ -106,9 +122,11 @@
       </visual>
     </link>
-  </macro>
+  </xacro:macro>
+  -->
   <!-- AngleBracket With USB Hub -->
-  <macro name="anglebracketusb" params="parent name *origin">
+  <!--
+  <xacro:macro name="anglebracketusb" params="parent name *origin">
     <joint name="${name}_joint" type="fixed">
-      <insert_block name="origin" />
+      <xacro:insert_block name="origin" />
       <parent link="${parent}"/>
       <child link="${name}_link" />
@@ -129,9 +147,11 @@
       </visual>
     </link>
-  </macro>
+  </xacro:macro>
+  -->
   <!-- KINECT -->
-  <macro name="kinect" params="parent name color llimit ulimit vlimit *origin">
+  <!--
+  <xacro:macro name="kinect" params="parent name color llimit ulimit vlimit *origin">
     <joint name="${name}_joint" type="revolute">
-      <insert_block name="origin" />
+      <xacro:insert_block name="origin" />
       <axis xyz="0 1 0"/>
       <limit effort="30" velocity="${vlimit}" lower="${llimit}" upper="${ulimit}" />
@@ -161,4 +181,5 @@
       </collision>
     </link>
-  </macro>
+  </xacro:macro>
+  -->
 </robot>

Commit message: UWB Position angepasst.

File: urdf/robotino.urdf (robot description, URDF)
Before this commit: robot robotino, 6 links, 5 joints
Joints:
- joint uwb_reciever_joint: origin xyz=0.05 0 0.15 rpy=0 0 0 -> xyz=0.04 0 0.26 rpy=0 0 0

File: urdf/robotino_body.xacro (robot description, xacro)
@@ -62,5 +62,5 @@
     </xacro:laser>
     <xacro:uwb name="uwb_reciever" parent="base_link">
-      <origin xyz="0.05 0 0.15" rpy="0 0 0"/>
+      <origin xyz="0.04 0 0.26" rpy="0 0 0"/>
     </xacro:uwb>
   </xacro:macro>
